Commit message: Velodyne added to husky. Can take up to 30 sec to spawn in Gazebo

File: urdf/husky.urdf.xacro (robot description, xacro)
@@ -28,4 +28,5 @@
   <xacro:include filename="$(find husky_description)/urdf/accessories/sick_lms1xx_mount.urdf.xacro"/>
   <xacro:include filename="$(find husky_description)/urdf/accessories/sensor_arch.urdf.xacro"/>
+  <xacro:include filename="$(find velodyne_description)/urdf/VLP-16.urdf.xacro"/>
   <xacro:include filename="$(find ur_description)/urdf/ur5.urdf.xacro" />
   <xacro:include filename="$(find husky_description)/urdf/accessories/gripper.urdf.xacro"/>
@@ -127,10 +128,9 @@
     </xacro:if>
     <xacro:if value="$(arg laser_enabled)">
+      <!-- Spawn laser scanner -->
       <sick_lms1xx_mount prefix="base" topic="scan"/>
       <joint name="laser_mount_joint" type="fixed">
-        <origin xyz="$(optenv HUSKY_LMS1XX_XYZ 0.8206 0.0 -0.20635)"
+        <origin xyz="$(optenv HUSKY_LMS1XX_XYZ 0.2206 0.0 0.00635)"
                 rpy="$(optenv HUSKY_LMS1XX_RPY 0.0 0.0 0.0)" />
-        <!-- <origin xyz="$(optenv HUSKY_LMS1XX_XYZ 0.2206 0.0 0.00635)"
-                rpy="$(optenv HUSKY_LMS1XX_RPY 0.0 0.0 0.0)" /> -->
         <parent link="top_plate_link" />
         <child link="base_laser_mount" />
@@ -138,4 +138,5 @@
     </xacro:if>
     <xacro:if value="$(arg kinect_enabled)">
+      <!-- Spawn kinect -->
       <xacro:sensor_arch prefix="" parent="top_plate_link">
         <origin xyz="-0.35 0 0.51" rpy="0 0 -3.14"/>
@@ -149,12 +150,7 @@
     </xacro:if>
     <xacro:if value="$(arg velodyne_enabled)">
-      <!--
-      <VLP-16 parent="camera_link" name="velodyne" topic="/velodyne_points">
-        <origin xyz="0 0 0.4" rpy="0 0 0" />
-      </VLP-16>
-      -->
-      <xacro:include filename="$(find velodyne_description)/urdf/VLP-16.urdf.xacro"/>
+      <!-- Spawn velodyne -->
       <VLP-16 parent="base_link" name="velodyne" topic="/velodyne_points">
-        <origin xyz="0 0 1" rpy="0 0 0" />
+        <origin xyz="-0.25 0 0.83" rpy="0 0 0" />
       </VLP-16>
     </xacro:if>
