Commit message: Re-enabled gps plugin and increased mass of husky

File: urdf/husky/husky.gazebo.xacro (robot description, xacro)
@@ -38,5 +38,4 @@
       </plugin>
     </gazebo>
-    <!--
     <gazebo>
       <plugin name="gps_controller" filename="libhector_gazebo_ros_gps.so">
@@ -47,6 +46,6 @@
         <topicName>navsat/fix</topicName>
         <velocityTopicName>navsat/vel</velocityTopicName>
-        <referenceLatitude>49.9</referenceLatitude>
-        <referenceLongitude>8.9</referenceLongitude>
+        <referenceLatitude>24.4793194</referenceLatitude>
+        <referenceLongitude>54.6105446</referenceLongitude>
         <referenceHeading>0</referenceHeading>
         <referenceAltitude>0</referenceAltitude>
@@ -54,5 +53,4 @@
       </plugin>
     </gazebo>
-    -->
     <xacro:if value="$(arg ur5_enabled)">
       <!--Remove when https://github.com/ros-industrial/universal_robot/pull/168 is resolved -->

File: urdf/husky/husky.urdf.xacro (robot description, xacro)
@@ -78,5 +78,5 @@
     <link name="inertial_link">
       <inertial>
-        <mass value="33.455" />
+        <mass value="53.455" />
         <origin xyz="-0.08748 -0.00085 0.09947" />
         <inertia ixx="0.6022" ixy="-0.02364" ixz="-0.1197" iyy="1.7386" iyz="-0.001544" izz="2.0296" />
