Commit message: Moved husky urdf files to folder, added GPS

File: urdf/husky/description.gazebo.xacro (robot description, xacro)
@@ -27,5 +27,5 @@
   <xacro:arg name="ur5_enabled" default="false" />
   <xacro:arg name="gripper_enabled" default="false" />
-  <xacro:include filename="$(find kuri_mbzirc_sim)/urdf/husky.urdf.xacro" />
+  <xacro:include filename="$(find kuri_mbzirc_sim)/urdf/husky/husky.urdf.xacro" />
   <xacro:include filename="$(find husky_gazebo)/urdf/husky.gazebo.xacro" />
   <!-- Gazebo plugin for ROS Control -->

File: urdf/husky/husky.urdf.xacro (robot description, xacro)
@@ -131,5 +131,5 @@
       <sick_lms1xx_mount prefix="base" topic="scan"/>
       <joint name="laser_mount_joint" type="fixed">
-        <origin xyz="$(optenv HUSKY_LMS1XX_XYZ 0.2206 0.0 0.00635)"
+        <origin xyz="$(optenv HUSKY_LMS1XX_XYZ 0.4 0.0 -0.20635)"
                 rpy="$(optenv HUSKY_LMS1XX_RPY 0.0 0.0 0.0)" />
         <parent link="top_plate_link" />

File: urdf/iris/iris_with_sensors.xacro (robot description, xacro)
@@ -128,3 +128,19 @@
     <origin xyz="0.0 0.0 -0.045" rpy="0 ${M_PI/2} 0"/>
   </xacro:generic_camera>
+  <!-- GPS -->
+  <gazebo>
+    <plugin name="gps_controller" filename="libhector_gazebo_ros_gps.so">
+      <updateRate>40</updateRate>
+      <robotNamespace>/</robotNamespace>
+      <bodyName>base_link</bodyName>
+      <frameId>base_link</frameId>
+      <topicName>navsat/fix</topicName>
+      <velocityTopicName>navsat/vel</velocityTopicName>
+      <referenceLatitude>49.9</referenceLatitude>
+      <referenceLongitude>8.9</referenceLongitude>
+      <referenceHeading>0</referenceHeading>
+      <referenceAltitude>0</referenceAltitude>
+      <drift>0.0001 0.0001 0.0001</drift>
+    </plugin>
+  </gazebo>
 </robot>

Commit message: Added webcam to simulate softkinetic

File: urdf/husky/description.gazebo.xacro (robot description, xacro)
@@ -27,4 +27,5 @@
   <xacro:arg name="ur5_enabled" default="false" />
   <xacro:arg name="gripper_enabled" default="false" />
+  <xacro:arg name="softkinetic_enabled" default="false" />
   <xacro:include filename="$(find kuri_mbzirc_sim)/urdf/husky/husky.urdf.xacro" />
   <xacro:include filename="$(find kuri_mbzirc_sim)/urdf/husky/husky.gazebo.xacro" />

File: urdf/husky/husky.gazebo.xacro (robot description, xacro)
@@ -23,4 +23,5 @@
 <robot name="husky_robot_gazebo" xmlns:xacro="http://ros.org/wiki/xacro">
   <xacro:include filename="$(find kuri_mbzirc_sim)/urdf/husky/accessories/kinect_camera.gazebo.xacro"/>
+  <xacro:include filename="$(find kuri_mbzirc_sim)/urdf/husky/accessories/softkinetic_camera.gazebo.xacro"/>
   <xacro:macro name="husky_robot_gazebo">
     <gazebo>
@@ -76,4 +77,7 @@
         <selfCollide>true</selfCollide>
       </gazebo>
+      <xacro:if value="$(arg softkinetic_enabled)">
+        <xacro:softkinetic_enabled prefix="camera2"/>
+      </xacro:if>
     </xacro:if>
     <xacro:if value="$(arg kinect_enabled)">

File: urdf/husky/husky.urdf.xacro (robot description, xacro)
@@ -127,4 +127,10 @@
         <xacro:pr2_gripper_simple_transmission />
       </xacro:if>
+      <xacro:if value="$(arg softkinetic_enabled)">
+        <!-- Spawn softkinetic -->
+        <xacro:softkinetic_camera_gazebo prefix="camera2" parent_link="ur5_arm_wrist_3_link">
+          <origin xyz="0 0.095 0.015" rpy="${M_PI} 0 ${M_PI/2}" />
+        </xacro:softkinetic_camera_gazebo>
+      </xacro:if>
     </xacro:if>
     <xacro:if value="$(arg laser_enabled)">
