Commit message: Copied SICK laser urdf from the lms1xx package for modification

File: urdf/husky/husky.urdf.xacro (robot description, xacro)
@@ -26,5 +26,5 @@
   <xacro:include filename="$(find husky_description)/urdf/wheel.urdf.xacro" />
   <xacro:include filename="$(find husky_description)/urdf/accessories/kinect_camera.urdf.xacro"/>
-  <xacro:include filename="$(find husky_description)/urdf/accessories/sick_lms1xx_mount.urdf.xacro"/>
+  <xacro:include filename="$(find kuri_mbzirc_sim)/urdf/husky/sick_lms1xx.urdf.xacro" />
   <xacro:include filename="$(find husky_description)/urdf/accessories/sensor_arch.urdf.xacro"/>
   <xacro:include filename="$(find velodyne_description)/urdf/VLP-16.urdf.xacro"/>
@@ -129,10 +129,10 @@
     <xacro:if value="$(arg laser_enabled)">
       <!-- Spawn laser scanner -->
-      <sick_lms1xx_mount prefix="base" topic="scan"/>
-      <joint name="laser_mount_joint" type="fixed">
-        <origin xyz="$(optenv HUSKY_LMS1XX_XYZ 0.4 0.0 -0.20635)"
+      <sick_lms1xx frame="base_laser" topic="scan"/>
+      <joint name="laser_joint" type="fixed">
+        <origin xyz="$(optenv HUSKY_LMS1XX_XYZ 0.38 0.0 -0.03135)"
                 rpy="$(optenv HUSKY_LMS1XX_RPY 0.0 0.0 0.0)" />
         <parent link="top_plate_link" />
-        <child link="base_laser_mount" />
+        <child link="base_laser" />
       </joint>
     </xacro:if>

Commit message: modified the wrenches ambient and tilted the kinect upward

File: urdf/husky/husky.urdf.xacro (robot description, xacro)
@@ -144,5 +144,5 @@
       </xacro:sensor_arch>
       <joint name="kinect_frame_joint" type="fixed">
-        <origin xyz="$(optenv HUSKY_KINECT_XYZ 0 0 0)" rpy="$(optenv HUSKY_KINECT_RPY 0 0.18 3.14)" />
+        <origin xyz="$(optenv HUSKY_KINECT_XYZ 0 0 0)" rpy="$(optenv HUSKY_KINECT_RPY 0 0 3.14)" />
         <parent link="sensor_arch_mount_link"/>
         <child link="camera_link"/>

Commit message: Corrected camera orientation

File: urdf/husky/husky.urdf.xacro (robot description, xacro)
@@ -130,5 +130,5 @@
         <!-- Spawn softkinetic -->
         <xacro:softkinetic_camera_gazebo prefix="camera2" parent_link="ur5_arm_wrist_3_link">
-          <origin xyz="0 0.095 0.015" rpy="${M_PI} 0 ${M_PI/2}" />
+          <origin xyz="0 0.095 0.015" rpy="0 0 ${M_PI/2}" />
         </xacro:softkinetic_camera_gazebo>
       </xacro:if>
