Commit message: added ground truth for the drone

File: urdf/iris/iris_with_sensors.urdf (robot description, URDF)
Before this commit: robot iris, 14 links, 13 joints
Links:
- added link /ground_truth/odometry_sensorgt_link, mass 1e-05
- added link /imugt_link, mass 1e-05
Joints:
- added joint /ground_truth/odometry_sensorgt_joint: type revolute, parent base_link, child /ground_truth/odometry_sensorgt_link, origin xyz=0.0 0.0 0.0 rpy=0.0 0.0 0.0, limit lower=0 upper=0 effort=0 velocity=0
- added joint /imugt_joint: type revolute, parent base_link, child /imugt_link, origin xyz=0 0 0 rpy=0 0 0, limit lower=0 upper=0 effort=0 velocity=0

File: urdf/iris/iris_with_sensors.xacro (robot description, xacro)
@@ -10,5 +10,5 @@
   <xacro:arg name='enable_mavlink_interface' default='true' />
   <xacro:arg name='enable_wind' default='false' />
-  <xacro:arg name='enable_ground_truth' default='false' />
+  <xacro:arg name='enable_ground_truth' default='true' />
   <xacro:arg name='enable_logging' default='false' />
   <xacro:arg name='log_file' default='iris' />
@@ -128,3 +128,19 @@
     <origin xyz="0.0 0.0 -0.045" rpy="0 ${M_PI/2} 0"/>
   </xacro:generic_camera>
+  <!-- GPS -->
+  <gazebo>
+    <plugin name="gps_controller" filename="libhector_gazebo_ros_gps.so">
+      <updateRate>40</updateRate>
+      <robotNamespace>/</robotNamespace>
+      <bodyName>base_link</bodyName>
+      <frameId>base_link</frameId>
+      <topicName>navsat/fix</topicName>
+      <velocityTopicName>navsat/vel</velocityTopicName>
+      <referenceLatitude>49.9</referenceLatitude>
+      <referenceLongitude>8.9</referenceLongitude>
+      <referenceHeading>0</referenceHeading>
+      <referenceAltitude>0</referenceAltitude>
+      <drift>0.0001 0.0001 0.0001</drift>
+    </plugin>
+  </gazebo>
 </robot>
